File: avr-carrier.kicad_pcb (KiCad board)
At the start: 2 copper layers, 71.5 x 71.5 mm, 0 parts

Commit message: stuff
Other:
- board text added: "${DATE} ${TEST}"
- board text added: "${TEST}"
- board text removed: "${date} ${test}"
Changed lines of the file:
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@@
   (net 0 "")
   (gr_rect (start 93.4 69.8) (end 164.9 141.3) (layer "Edge.Cuts") (width 0.1) (fill none))
-  (gr_text "${date}\n\n${test}" (at 128.3 100.7) (layer "F.SilkS")
+  (gr_text "${DATE}\n\n${TEST}" (at 128.3 100.7) (layer "F.SilkS")
     (effects (font (size 2 2) (thickness 0.15)))
   )
+  (gr_text "${TEST}" (at 122.4 124.4) (layer "F.SilkS")
+    (effects (font (size 1 1) (thickness 0.15)))
+  )
   (zone (net 0) (net_name "") (layer "F.Cu") (hatch edge 0.508)

Commit message: stuff
Other:
- board text added: "${test}"
- board text added: "${version}"
- board text removed: "${DATE} ${TEST}"
- board text removed: "${TEST}"
Changed lines of the file:
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@@
   (net 0 "")
   (gr_rect (start 93.4 69.8) (end 164.9 141.3) (layer "Edge.Cuts") (width 0.1) (fill none))
-  (gr_text "${DATE}\n\n${TEST}" (at 128.3 100.7) (layer "F.SilkS")
+  (gr_text "${version}" (at 114.7 85.1) (layer "F.SilkS")
     (effects (font (size 2 2) (thickness 0.15)))
   )
-  (gr_text "${TEST}" (at 122.4 124.4) (layer "F.SilkS")
+  (gr_text "${test}" (at 115.9 113.2) (layer "F.SilkS")
     (effects (font (size 1 1) (thickness 0.15)))
   )

Commit message: stuff
Other:
- board text added: "${date}"
Changed lines of the file:
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@@
+    (effects (font (size 1 1) (thickness 0.15)))
+  )
+  (gr_text "${date}" (at 135 101.3) (layer "F.SilkS")
     (effects (font (size 1 1) (thickness 0.15)))
   )

Commit message: init
Parts:
- added C1: 860020372001, 860020372001:CAPPRD200W52D500H1250, F.Cu at (120.0, 117.0)
- added D1: LED, LTL-4232:LTL4232, F.Cu at (158.4, 81.2)
- added D2: LED, LTL-4232:LTL4232, F.Cu at (158.4, 116.3)
- added G***: LOGO, library:one, B.Cu at (135.0, 90.1)
- added J1: Conn_01x10, Connector_PinHeader_2.54mm:PinHeader_1x10_P2.54mm_Vertical, B.Cu at (132.5, 74.6)
- added J2: Conn_01x08, Connector_PinHeader_2.54mm:PinHeader_1x08_P2.54mm_Vertical, B.Cu at (136.5, 122.9)
- added J3: 24-3553-10, 24-3553-10:24355310, F.Cu at (121.8, 94.9)
- added J4: Conn_01x08, Connector_PinHeader_2.54mm:PinHeader_1x08_P2.54mm_Vertical, B.Cu at (154.3, 74.6)
- added J5: Conn_01x06, Connector_PinHeader_2.54mm:PinHeader_1x06_P2.54mm_Vertical, B.Cu at (154.3, 122.9)
- added R1: 100k, CFR-12JR-52-300R:RESAD1100W50L340D190, F.Cu at (152.8, 81.2)
- added R2: 100k, CFR-12JR-52-300R:RESAD1100W50L340D190, F.Cu at (152.8, 116.3)
Routing:
- net (no net): track 0.00 -> 259.3 mm
- added copper zone on B.Cu, net (none)
- removed copper zone on F.Cu, net (none)
Other:
- board size 71.5 x 71.5 mm -> 55.6 x 53.3 mm
- board text added: "+"
- board text added: "-"
- board text removed: "${date}"
- board text removed: "${test}"
- board text removed: "${version}"

Commit message: fix everything
Parts:
- C1: footprint 860020372001:CAPPRD200W52D500H1250 -> CC_Capacitors:CAPPRD200W52D500H1250
- D1, D2: footprint LTL-4232:LTL4232 -> CC_LEDs:LTL4232
- J1: value Conn_01x10 -> Conn_01x08; footprint Connector_PinHeader_2.54mm:PinHeader_1x10_P2.54mm_Vertical -> Connector_PinHeader_2.54mm:PinHeader_1x08_P2.54mm_Vertical
- J3: value 24-3553-10 -> Conn_01x10; footprint 24-3553-10:24355310 -> Connector_PinHeader_2.54mm:PinHeader_1x10_P2.54mm_Vertical; moved to B.Cu
- J4: value Conn_01x08 -> 24-3553-10; footprint Connector_PinHeader_2.54mm:PinHeader_1x08_P2.54mm_Vertical -> CC_Misc:24355310; moved to F.Cu
- R1, R2: footprint CFR-12JR-52-300R:RESAD1100W50L340D190 -> CC_Resistors:RESAD1100W50L340D190
- moved J4 38.3 mm to (121.8, 94.9), turned to 0 degrees
- moved J3 22.9 mm to (132.4, 74.6), turned to 90 degrees
- moved J1 21.8 mm to (154.3, 74.6)
- moved G*** 20.0 mm to (133.7, 110.1)
- moved R2 0.11 mm to (152.7, 116.2)
Connections:
- C1 pad 1: (no net) -> Net-(C1-Pad1)
- C1 pad 2: (no net) -> GND
- D1 pad 1: (no net) -> GND
- D1 pad 2: (no net) -> Net-(D1-Pad2)
- D2 pad 1: (no net) -> GND
- D2 pad 2: (no net) -> Net-(D2-Pad2)
- J1 pad 1: (no net) -> unconnected-(J1-Pad1)
- J1 pad 2: (no net) -> unconnected-(J1-Pad2)
- J1 pad 3: (no net) -> unconnected-(J1-Pad3)
- J1 pad 4: (no net) -> unconnected-(J1-Pad4)
- J1 pad 5: (no net) -> unconnected-(J1-Pad5)
- J1 pad 6: (no net) -> unconnected-(J1-Pad6)
- J1 pad 7: (no net) -> unconnected-(J1-Pad7)
- J1 pad 8: (no net) -> unconnected-(J1-Pad8)
- J2 pad 1: (no net) -> unconnected-(J2-Pad1)
- J2 pad 2: (no net) -> GND
- J2 pad 3: (no net) -> GND
- J2 pad 4: (no net) -> +5V
- J2 pad 5: (no net) -> unconnected-(J2-Pad5)
- J2 pad 6: (no net) -> Net-(C1-Pad1)
- J2 pad 7: (no net) -> unconnected-(J2-Pad7)
- J2 pad 8: (no net) -> unconnected-(J2-Pad8)
- J3 pad 1: (no net) -> unconnected-(J3-Pad1)
- J3 pad 10: (no net) -> unconnected-(J3-Pad10)
- J3 pad 2: (no net) -> unconnected-(J3-Pad2)
- J3 pad 3: (no net) -> Net-(J3-Pad3)
- J3 pad 4: (no net) -> Net-(J3-Pad4)
- J3 pad 5: (no net) -> Net-(J3-Pad5)
- J3 pad 6: (no net) -> Net-(J3-Pad6)
- J3 pad 7: (no net) -> GND
- J3 pad 8: (no net) -> unconnected-(J3-Pad8)
- J3 pad 9: (no net) -> unconnected-(J3-Pad9)
- J4 pad 1: (no net) -> unconnected-(J4-Pad1)
- J4 pad 2: (no net) -> unconnected-(J4-Pad2)
- J4 pad 3: (no net) -> unconnected-(J4-Pad3)
- J4 pad 4: (no net) -> unconnected-(J4-Pad4)
- J4 pad 5: (no net) -> unconnected-(J4-Pad5)
- J4 pad 6: (no net) -> unconnected-(J4-Pad6)
- J4 pad 7: (no net) -> unconnected-(J4-Pad7)
- J4 pad 8: (no net) -> unconnected-(J4-Pad8)
- J5 pad 1: (no net) -> unconnected-(J5-Pad1)
- J5 pad 2: (no net) -> unconnected-(J5-Pad2)
- J5 pad 3: (no net) -> unconnected-(J5-Pad3)
- J5 pad 4: (no net) -> unconnected-(J5-Pad4)
- J5 pad 5: (no net) -> unconnected-(J5-Pad5)
- J5 pad 6: (no net) -> unconnected-(J5-Pad6)
- R1 pad 1: (no net) -> Net-(D1-Pad2)
- R1 pad 2: (no net) -> Net-(J3-Pad5)
- R2 pad 1: (no net) -> Net-(D2-Pad2)
- R2 pad 2: (no net) -> Net-(J3-Pad4)
Routing:
- net (no net): track 259.3 -> 0.00 mm
- net Net-(J3-Pad4): track 0.00 -> 59.5 mm
- net +5V: track 0.00 -> 52.5 mm
- net Net-(J3-Pad5): track 0.00 -> 49.1 mm
- net Net-(J3-Pad3): track 0.00 -> 46.3 mm
- net Net-(J3-Pad6): track 0.00 -> 33.1 mm
- net Net-(C1-Pad1): track 0.00 -> 8.46 mm
- net Net-(D2-Pad2): track 0.00 -> 3.05 mm
- net Net-(D1-Pad2): track 0.00 -> 3.05 mm
- added copper zone on B.Cu, net GND
- removed copper zone on B.Cu, net (none)
Other:
- board text added: "${version}"
