File: avr-carrier.kicad_pcb (KiCad board)
At the start: 2 copper layers, 55.6 x 53.3 mm, 11 parts, among them J1 Conn_01x08, J2 Conn_01x08, J3 Conn_01x10, J4 24-3553-10, J5 Conn_01x06

Commit message: slight fixing
Parts:
- renumbered J4 to J1
Changed lines of the file:
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@@
     (property "Sheetname" "")
     (attr through_hole)
-    (fp_text reference "J4" (at 12 3.81) (layer "F.SilkS")
+    (fp_text reference "J1" (at 12 3.81) (layer "F.SilkS")
       (effects (font (size 1.27 1.27) (thickness 0.254)))
     )
@@
     (property "Sheetname" "")
     (attr through_hole)
-    (fp_text reference "J3" (at 0.1 -25 90) (layer "B.SilkS")
+    (fp_text reference "J3" (at 0.1 -25.3 90) (layer "B.SilkS")
       (effects (font (size 1 1) (thickness 0.15)) (justify mirror))
     )
@@
     (property "Sheetname" "")
     (attr through_hole)
-    (fp_text reference "J5" (at 0 2.33 90) (layer "B.SilkS")
+    (fp_text reference "J5" (at 0 2.486 90) (layer "B.SilkS")
       (effects (font (size 1 1) (thickness 0.15)) (justify mirror))
     )
@@
     (property "Sheetname" "")
     (attr through_hole)
-    (fp_text reference "J2" (at 0 2.33 90) (layer "B.SilkS")
+    (fp_text reference "J2" (at 0.06 -20.334 90) (layer "B.SilkS")
       (effects (font (size 1 1) (thickness 0.15)) (justify mirror))
     )
