File: avr-carrier.kicad_sch (KiCad schematic)
At the start: 10 parts, among them J1 Conn_01x08, J2 Conn_01x08, J3 Conn_01x10, J4 24-3553-10, J5 Conn_01x06

Commit message: fix everything
Parts:
- removed J4: 24-3553-10, 24-3553-10:24355310, symbol avr_programmer-rescue:24-3553-10-24-3553-10
- added J4: 24-3553-10, CC_Misc:24355310, symbol CC_Misc:24-3553-10
- C1: footprint 860020372001:CAPPRD200W52D500H1250 -> CC_Capacitors:CAPPRD200W52D500H1250
- D1, D2: footprint LTL-4232:LTL4232 -> CC_LEDs:LTL4232
- R1, R2: footprint CFR-12JR-52-300R:RESAD1100W50L340D190 -> CC_Resistors:RESAD1100W50L340D190
Connections:
- net +5V: now also J4.17
- net GND: now also J4.24
- net at J3.3 (Pin_3): now also J4.18
- net at J3.6 (Pin_6): now also J4.19
- net at J3.5 (Pin_5), R1.2: now also J4.21
- net at J3.4 (Pin_4), R2.2: now also J4.23

Commit message: fix rules
Parts:
- C1: symbol avr_programmer-rescue:860020372001-860020372001 -> CC_Capacitors:860020372001
Connections:
- no-connect marks 0 -> 43
Changed lines of the file:
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@@
   (junction (at 181.61 77.47) (diameter 0) (color 0 0 0 0)
   )
+  (no_connect (at 189.23 92.71))
+  (no_connect (at 109.22 123.19))
+  (no_connect (at 101.6 123.19))
+  (no_connect (at 116.84 87.63))
+  (no_connect (at 163.83 80.01))
+  (no_connect (at 153.67 125.73))
+  (no_connect (at 156.21 105.41))
+  (no_connect (at 168.91 80.01))
+  (no_connect (at 179.07 105.41))
+  (no_connect (at 85.09 81.28))
+  (no_connect (at 171.45 80.01))
+  (no_connect (at 158.75 105.41))
+  (no_connect (at 158.75 80.01))
+  (no_connect (at 151.13 125.73))
+  (no_connect (at 143.51 125.73))
+  (no_connect (at 163.83 105.41))
+  (no_connect (at 171.45 105.41))
+  (no_connect (at 156.21 125.73))
+  (no_connect (at 148.59 125.73))
+  (no_connect (at 161.29 80.01))
+  (no_connect (at 82.55 81.28))
+  (no_connect (at 146.05 92.71))
+  (no_connect (at 95.25 81.28))
+  (no_connect (at 114.3 87.63))
+  (no_connect (at 153.67 105.41))
+  (no_connect (at 166.37 105.41))
+  (no_connect (at 119.38 87.63))
+  (no_connect (at 87.63 81.28))
+  (no_connect (at 137.16 87.63))
+  (no_connect (at 104.14 123.19))
+  (no_connect (at 168.91 105.41))
+  (no_connect (at 166.37 80.01))
+  (no_connect (at 92.71 81.28))
+  (no_connect (at 176.53 105.41))
+  (no_connect (at 90.17 81.28))
+  (no_connect (at 156.21 80.01))
+  (no_connect (at 146.05 125.73))
+  (no_connect (at 134.62 87.63))
+  (no_connect (at 119.38 123.19))
+  (no_connect (at 100.33 81.28))
+  (no_connect (at 97.79 81.28))
+  (no_connect (at 153.67 80.01))
+  (no_connect (at 161.29 105.41))
   (wire (pts (xy 198.12 54.61) (xy 198.12 57.15))
     (stroke (width 0) (type default) (color 0 0 0 0))
@@
     (stroke (width 0) (type default) (color 0 0 0 0))
   )
-  (wire (pts (xy 116.84 121.92) (xy 116.84 123.19))
-    (stroke (width 0) (type default) (color 0 0 0 0))
-  )
-  (wire (pts (xy 114.3 121.92) (xy 114.3 123.19))
+  (wire (pts (xy 116.84 119.38) (xy 116.84 123.19))
+    (stroke (width 0) (type default) (color 0 0 0 0))
+  )
+  (wire (pts (xy 114.3 119.38) (xy 114.3 123.19))
     (stroke (width 0) (type default) (color 0 0 0 0))
   )
@@
     (stroke (width 0) (type default) (color 0 0 0 0))
   )
+  (wire (pts (xy 90.17 66.04) (xy 90.17 71.12))
+    (stroke (width 0) (type default) (color 0 0 0 0))
+  )
   (wire (pts (xy 142.24 111.76) (xy 173.99 111.76))
     (stroke (width 0) (type default) (color 0 0 0 0))
@@
     (stroke (width 0) (type default) (color 0 0 0 0))
   )
-  (wire (pts (xy 111.76 121.92) (xy 111.76 123.19))
+  (wire (pts (xy 111.76 119.38) (xy 111.76 123.19))
     (stroke (width 0) (type default) (color 0 0 0 0))
   )
@@
   )
   (wire (pts (xy 179.07 74.93) (xy 179.07 80.01))
+    (stroke (width 0) (type default) (color 0 0 0 0))
+  )
+  (wire (pts (xy 101.6 66.04) (xy 101.6 71.12))
     (stroke (width 0) (type default) (color 0 0 0 0))
   )
@@
     (pin "2")
   )
+  (symbol (lib_id "power:PWR_FLAG") (at 90.17 71.12 180) (unit 1)
+    (in_bom yes) (on_board yes) (fields_autoplaced)
+    (property "Reference" "#FLG_GND0101" (id 0) (at 90.17 73.025 0)
+      (effects (font (size 1.27 1.27)) hide)
+    )
+    (property "Value" "PWR_FLAG" (id 1) (at 90.17 75.5634 0))
+    (property "Footprint" "" (id 2) (at 90.17 71.12 0)
+      (effects (font (size 1.27 1.27)) hide)
+    )
+    (property "Datasheet" "~" (id 3) (at 90.17 71.12 0)
+      (effects (font (size 1.27 1.27)) hide)
+    )
+    (pin "1")
+  )
+  (symbol (lib_id "power:+5V") (at 101.6 66.04 0) (unit 1)
+    (in_bom yes) (on_board yes) (fields_autoplaced)
+    (property "Reference" "#PWR0110" (id 0) (at 101.6 69.85 0)
+      (effects (font (size 1.27 1.27)) hide)
+    )
+    (property "Value" "+5V" (id 1) (at 101.6 62.4642 0))
+    (property "Footprint" "" (id 2) (at 101.6 66.04 0)
+      (effects (font (size 1.27 1.27)) hide)
+    )
+    (property "Datasheet" "" (id 3) (at 101.6 66.04 0)
+      (effects (font (size 1.27 1.27)) hide)
+    )
+    (pin "1")
+  )
   (symbol (lib_id "power:GND") (at 181.61 107.95 0) (unit 1)
     (in_bom yes) (on_board yes)
@@
     (pin "1")
   )
-  (symbol (lib_id "power:GND") (at 114.3 121.92 180) (unit 1)
-    (in_bom yes) (on_board yes)
-    (property "Reference" "#PWR0108" (id 0) (at 114.3 115.57 0)
-      (effects (font (size 1.27 1.27)) hide)
-    )
-    (property "Value" "GND" (id 1) (at 115.57 116.84 0))
-    (property "Footprint" "" (id 2) (at 114.3 121.92 0)
-      (effects (font (size 1.27 1.27)) hide)
-    )
-    (property "Datasheet" "" (id 3) (at 114.3 121.92 0)
-      (effects (font (size 1.27 1.27)) hide)
-    )
-    (pin "1")
-  )
-  (symbol (lib_id "power:+5V") (at 111.76 121.92 0) (unit 1)
-    (in_bom yes) (on_board yes)
-    (property "Reference" "#PWR0109" (id 0) (at 111.76 125.73 0)
-      (effects (font (size 1.27 1.27)) hide)
-    )
-    (property "Value" "+5V" (id 1) (at 111.76 116.84 0))
-    (property "Footprint" "" (id 2) (at 111.76 121.92 0)
-      (effects (font (size 1.27 1.27)) hide)
-    )
-    (property "Datasheet" "" (id 3) (at 111.76 121.92 0)
+  (symbol (lib_id "power:GND") (at 114.3 119.38 180) (unit 1)
+    (in_bom yes) (on_board yes)
+    (property "Reference" "#PWR0108" (id 0) (at 114.3 113.03 0)
+      (effects (font (size 1.27 1.27)) hide)
+    )
+    (property "Value" "GND" (id 1) (at 115.57 114.3 0))
+    (property "Footprint" "" (id 2) (at 114.3 119.38 0)
+      (effects (font (size 1.27 1.27)) hide)
+    )
+    (property "Datasheet" "" (id 3) (at 114.3 119.38 0)
+      (effects (font (size 1.27 1.27)) hide)
+    )
+    (pin "1")
+  )
+  (symbol (lib_id "power:+5V") (at 111.76 119.38 0) (unit 1)
+    (in_bom yes) (on_board yes)
+    (property "Reference" "#PWR0109" (id 0) (at 111.76 123.19 0)
+      (effects (font (size 1.27 1.27)) hide)
+    )
+    (property "Value" "+5V" (id 1) (at 111.76 114.3 0))
+    (property "Footprint" "" (id 2) (at 111.76 119.38 0)
+      (effects (font (size 1.27 1.27)) hide)
+    )
+    (property "Datasheet" "" (id 3) (at 111.76 119.38 0)
       (effects (font (size 1.27 1.27)) hide)
     )
@@
     )
     (property "Datasheet" "" (id 3) (at 173.99 77.47 0)
+      (effects (font (size 1.27 1.27)) hide)
+    )
+    (pin "1")
+  )
+  (symbol (lib_id "power:GND") (at 90.17 66.04 180) (unit 1)
+    (in_bom yes) (on_board yes) (fields_autoplaced)
+    (property "Reference" "#PWR0111" (id 0) (at 90.17 59.69 0)
+      (effects (font (size 1.27 1.27)) hide)
+    )
+    (property "Value" "GND" (id 1) (at 90.17 62.4642 0))
+    (property "Footprint" "" (id 2) (at 90.17 66.04 0)
+      (effects (font (size 1.27 1.27)) hide)
+    )
+    (property "Datasheet" "" (id 3) (at 90.17 66.04 0)
       (effects (font (size 1.27 1.27)) hide)
     )
@@
     (pin "8")
     (pin "9")
+  )
+  (symbol (lib_id "power:PWR_FLAG") (at 101.6 71.12 180) (unit 1)
+    (in_bom yes) (on_board yes) (fields_autoplaced)
+    (property "Reference" "#FLG_5v0101" (id 0) (at 101.6 73.025 0)
+      (effects (font (size 1.27 1.27)) hide)
+    )
+    (property "Value" "PWR_FLAG" (id 1) (at 101.6 75.5634 0))
+    (property "Footprint" "" (id 2) (at 101.6 71.12 0)
+      (effects (font (size 1.27 1.27)) hide)
+    )
+    (property "Datasheet" "~" (id 3) (at 101.6 71.12 0)
+      (effects (font (size 1.27 1.27)) hide)
+    )
+    (pin "1")
   )
   (symbol (lib_id "CC_Misc:24-3553-10") (at 146.05 92.71 0) (unit 1)
@@
     (pin "MH2")
   )
-  (symbol (lib_id "avr_programmer-rescue:860020372001-860020372001") (at 91.44 116.84 180) (unit 1)
+  (symbol (lib_id "CC_Capacitors:860020372001") (at 91.44 116.84 180) (unit 1)
     (in_bom yes) (on_board yes)
     (property "Reference" "C1" (id 0) (at 85.09 110.0582 0))
@@
     (pin "2")
   )
-  (symbol (lib_id "power:GND") (at 116.84 121.92 180) (unit 1)
-    (in_bom yes) (on_board yes)
-    (property "Reference" "#PWR0107" (id 0) (at 116.84 115.57 0)
-      (effects (font (size 1.27 1.27)) hide)
-    )
-    (property "Value" "GND" (id 1) (at 119.38 116.84 0))
-    (property "Footprint" "" (id 2) (at 116.84 121.92 0)
-      (effects (font (size 1.27 1.27)) hide)
-    )
-    (property "Datasheet" "" (id 3) (at 116.84 121.92 0)
+  (symbol (lib_id "power:GND") (at 116.84 119.38 180) (unit 1)
+    (in_bom yes) (on_board yes)
+    (property "Reference" "#PWR0107" (id 0) (at 116.84 113.03 0)
+      (effects (font (size 1.27 1.27)) hide)
+    )
+    (property "Value" "GND" (id 1) (at 119.38 114.3 0))
+    (property "Footprint" "" (id 2) (at 116.84 119.38 0)
+      (effects (font (size 1.27 1.27)) hide)
+    )
+    (property "Datasheet" "" (id 3) (at 116.84 119.38 0)
       (effects (font (size 1.27 1.27)) hide)
     )
@@
   )
   (symbol_instances
+    (path "/c9d6fe12-53f5-4856-a032-20f09014ddce"
+      (reference "#FLG_5v0101") (unit 1) (value "PWR_FLAG") (footprint "")
+    )
+    (path "/509fecfa-874c-45ab-873b-e7ca9c51f2f8"
+      (reference "#FLG_GND0101") (unit 1) (value "PWR_FLAG") (footprint "")
+    )
     (path "/539c2212-7ffb-40d3-a670-94e793f677dc"
       (reference "#PWR0101") (unit 1) (value "GND") (footprint "")
@@
       (reference "#PWR0109") (unit 1) (value "+5V") (footprint "")
     )
+    (path "/530fbf9d-020c-48c1-a483-19f718379b09"
+      (reference "#PWR0110") (unit 1) (value "+5V") (footprint "")
+    )
+    (path "/96242899-6fa6-4fef-ac35-03f3194e31f3"
+      (reference "#PWR0111") (unit 1) (value "GND") (footprint "")
+    )
     (path "/cc76ce5e-402e-4efa-8268-ddd844c8bb12"
